Commit message: added example for force sensor

File: examples/sai2/02-fixed_joint/ppbot.urdf (robot description, URDF)
Before this commit: robot PBot, 3 links, 2 joints
Links:
- link link1: mass 1 -> 0.5; geometry collision sphere radius=0.1; visual sphere radius=0.1
Joints:
- joint j1: axis (none) -> 0 0 1; origin xyz=0.000000 0.000000 0.200000 rpy=-0.000000 0.000000 -0.000000 -> xyz=0.000000 0.201000 0.050000 rpy=-0.000000 0.000000 -0.000000; type fixed -> prismatic
