Commit message: added convenience functions to pause the simulation and get the simulated time

File: examples/sai2/02-fixed_joint/pbot_fixed_joint.urdf (robot description, URDF)
Before this commit: robot PBot_fixed_description, 3 links, 2 joints
Joints:
- joint j1: limit lower=-2.967 upper=2.967 effort=176 velocity=1.7104 -> (none)

File: examples/sai2/05-force_sensor/pbot.urdf (robot description, URDF)
Before this commit: robot PBot, 3 links, 2 joints
Joints:
- joint j_sensor: limit lower=-2.967 upper=2.967 effort=176 velocity=1.7104 -> (none)
