Commit message: added joint limit and damping (parsed from urdf file)

File: examples/sai2/03-spherical_joint/spherical_bot.urdf (robot description, URDF)
Before this commit: robot SphericalBot_description, 4 links, 3 joints
Joints:
- joint j0: limit lower=-2.967 upper=2.967 effort=176 velocity=1.7104 -> (none)
