Commit message: clean up logic of simulated force sensor

File: examples/sai2/05-force_sensor/pppbot.urdf (robot description, URDF)
Before this commit: robot PBot, 3 links, 2 joints
Links:
- added link link1, mass 0.01
- added link link2, mass 5; visual sphere radius=0.1
- link link0: mass 1 -> 0.01; geometry 
Joints:
- added joint j1: type prismatic, parent link0, child link1, origin xyz=0.000000 0.000000 0.000000 rpy=-0.000000 0.000000 -0.000000, axis 0 1 0, limit lower=-2.967 upper=2.967 effort=176 velocity=1.7104
- added joint j2: type prismatic, parent link1, child link2, origin xyz=0.000000 0.000000 0.000000 rpy=-0.000000 0.000000 -0.000000, axis 1 0 0, limit lower=-2.967 upper=2.967 effort=176 velocity=1.7104
- joint j_sensor: parent link0 -> link2
