Commit message: added support for continuous joints (revolute without limits) and for enabling/disabling joint limits in sim

File: examples/sai2/03-spherical_joint_and_ui_interactions/rrrbot.urdf (robot description, URDF)
Before this commit: robot RRRBot_description, 6 links, 5 joints
Joints:
- joint j0: limit lower=-2.967 upper=2.967 effort=176 velocity=1.7104 -> (none); type revolute -> continuous
- joint j1: limit lower=-2.967 upper=2.967 effort=176 velocity=1.7104 -> (none); type revolute -> continuous
- joint j2: limit lower=-2.967 upper=2.967 effort=176 velocity=1.7104 -> (none); type revolute -> continuous

File: examples/sai2/04-joint_limits_and_damping/rrbot.urdf (robot description, URDF)
Before this commit: robot RRBot_description, 3 links, 2 joints
Joints:
- joint j1: type continuous -> revolute
