Commit message: cleanup urdf parsing and examples

File: examples/04-joint_limits_and_damping/double_pendulum_jl_damping.urdf (robot description, URDF)
Before this commit: robot RRBot_description, 3 links, 2 joints
Joints:
- joint j0: limit lower=-2.967 upper=2.967 effort=176 velocity=1.7104 -> lower=0.3 upper=1.0 effort=176 velocity=1.7104
- joint j1: limit lower=-2.967 upper=2.967 effort=176 velocity=1.7104 -> lower=-0.1 upper=1.0 effort=176 velocity=1.7104
